File: Hardware/kicad_project/pcb/MainPCB_V2/MainPCB_V2.1.kicad_pcb (KiCad board)
At the start: 2 copper layers, 29 x 99 mm, 28 parts, among them J1 Conn_01x08, J2 Conn_01x08, J3 Power Input, J4 MCP4758 Board, J5 POWER IN, J6 Conn_01x07, J7 Conn_01x07, U1 MCP6004, U2 L7805

Commit message: Now the MCP4728 uses it's own I2C bus on separate pins
Parts:
- J3: value Power Input -> Power Jumper
Connections:
- J4 pad 3: SCL -> SCL2
- J4 pad 4: SDA -> SDA2
- J6 pad 7: unconnected-(J6-Pin_7-Pad7) -> SCL2
- J7 pad 1: unconnected-(J7-Pin_1-Pad1) -> SDA2
Routing:
- net SDA: track 78.0 -> 24.3 mm, vias 1 -> 0
- net SDA2: track 0.00 -> 52.2 mm
- net SCL: track 72.4 -> 24.5 mm
- net SCL2: track 0.00 -> 44.6 mm
